File: PWR_buck_12V_switcher.sch (KiCad schematic (older format))
At the start: 16 parts, among them Q1001 MOS_PRO, U1001 LM2596

Commit message: progress
Connections:
- wire segments 23 -> 22
Changed lines of the file:
@@
 LIBS:STM32F407IGT6
 LIBS:slc_oem
+LIBS:minefi-cache
 EELAYER 27 0
 EELAYER END
@@
 Sheet 5 6
 Title "Frankenso"
-Date "26 jul 2015"
+Date "28 jul 2015"
 Rev ".02"
 Comp "rusEFI.com"
@@
 OUT
 $Comp
-L GND #PWR047
-U 1 1 52C4D1EB
-P 7450 6900
-F 0 "#PWR047" H 7450 6900 30  0001 C CNN
-F 1 "GND" H 7450 6830 30  0001 C CNN
-F 2 "" H 7450 6900 60  0000 C CNN
-F 3 "" H 7450 6900 60  0000 C CNN
-	1    7450 6900
-	1    0    0    -1
-$EndComp
-Wire Wire Line
-	7450 6850 7450 6900
-$Comp
 L DIODE D1002
