File: minefi.sch (KiCad schematic (older format))
At the start: 21 parts, among them P11 CONN_1, P13 CONN_1, P16 CONN_1, P18 CONN_1, P20 CONN_1, P21 CONN_1, P23 CONN_1, P4 CONN_25, P5 CONN_3X2, P51 CONN_1, P52 CONN_1

Commit message: progress
Parts:
- removed P20, P21, P23: CONN_1, SIL-1, symbol CONN_1
Connections:
- net CAM+: now also P4.8 (P8); no longer P4.7 (P7)
- net CAM-: now also P4.7 (P7); no longer P4.8 (P8)
Changed lines of the file:
@@
 LIBS:STM32F407IGT6
 LIBS:slc_oem
+LIBS:minefi-cache
 EELAYER 27 0
 EELAYER END
@@
 Sheet 1 6
 Title "Frankenso"
-Date "26 jul 2015"
+Date "28 jul 2015"
 Rev ".04"
 Comp "rusEFI.com"
@@
 Text Label 12500 2550 3    60   ~ 0
 LOW-1A-01_2
+Text Label 14250 2100 3    60   ~ 0
+CAM+
 Text Label 14150 2100 3    60   ~ 0
-CAM+
-Text Label 14250 2100 3    60   ~ 0
 CAM-
 Text Label 14050 2100 3    60   ~ 0
@@
 	-1   0    0    1
 $EndComp
-$Comp
-L CONN_1 P20
-U 1 1 53BC309C
-P 9250 4400
-F 0 "P20" H 9330 4400 40  0000 L CNN
-F 1 "CONN_1" H 9250 4455 30  0001 C CNN
-F 2 "SIL-1" V 2780 -1900 60  0001 C CNN
-F 3 "" H 9250 4400 60  0001 C CNN
-F 4 "DO NOT POPULATE,DNP" V 2780 -1900 60  0001 C CNN "mfg,mfg#"
-F 5 "DO NOT POPULATE,DNP" V 2780 -1900 60  0001 C CNN "vend1,vend1#"
-	1    9250 4400
-	1    0    0    -1
-$EndComp
-$Comp
-L CONN_1 P21
-U 1 1 53BC30A2
-P 9250 4700
-F 0 "P21" H 9330 4700 40  0000 L CNN
-F 1 "CONN_1" H 9250 4755 30  0001 C CNN
-F 2 "SIL-1" V 2780 -1700 60  0001 C CNN
-F 3 "" H 9250 4700 60  0001 C CNN
-F 4 "DO NOT POPULATE,DNP" V 2780 -1700 60  0001 C CNN "mfg,mfg#"
-F 5 "DO NOT POPULATE,DNP" V 2780 -1700 60  0001 C CNN "vend1,vend1#"
-	1    9250 4700
-	1    0    0    -1
-$EndComp
-$Comp
-L CONN_1 P23
-U 1 1 53BC30AE
-P 9250 4000
-F 0 "P23" H 9330 4000 40  0000 L CNN
-F 1 "CONN_1" H 9250 4055 30  0001 C CNN
-F 2 "SIL-1" V 1130 2600 60  0001 C CNN
-F 3 "" H 9250 4000 60  0001 C CNN
-F 4 "DO NOT POPULATE,DNP" V 1130 2600 60  0001 C CNN "mfg,mfg#"
-F 5 "DO NOT POPULATE,DNP" V 1130 2600 60  0001 C CNN "vend1,vend1#"
-	1    9250 4000
-	1    0    0    -1
-$EndComp
 NoConn ~ 7750 7700
 NoConn ~ 7750 7600
@@
 	1    0    0    -1
 $EndComp
-Text Label 5700 5250 2    60   ~ 0
-5V
 NoConn ~ 7750 10000
 $Sheet
@@
 Wire Wire Line
 	7600 6400 7750 6400
-Connection ~ 9100 4750
-Wire Wire Line
-	9100 4700 9100 4750
-Connection ~ 9100 4450
-Wire Wire Line
-	9100 4400 9100 4450
-Connection ~ 9100 4050
-Wire Wire Line
-	9100 4000 9100 4050
 Wire Wire Line
 	9450 6800 9600 6800
@@
 	7150 4150 7750 4150
 Wire Wire Line
-	9000 4950 9600 4950
-Wire Wire Line
-	9000 4850 9600 4850
-Wire Wire Line
-	9000 4750 9600 4750
-Wire Wire Line
-	9000 4250 9600 4250
-Wire Wire Line
 	9000 4150 9600 4150
 Wire Wire Line
@@
 Wire Wire Line
 	9000 3950 9600 3950
-Wire Wire Line
-	9000 4650 9600 4650
-Wire Wire Line
-	9000 4550 9600 4550
-Wire Wire Line
-	9000 4450 9600 4450
-Wire Wire Line
-	9000 4350 9600 4350
 Wire Wire Line
 	9000 3850 9600 3850
@@
 NoConn ~ 11100 4850
 NoConn ~ 11100 4950
+Text Label 5700 5250 2    60   ~ 0
+5V
+Wire Wire Line
+	9000 4250 9600 4250
 $EndSCHEMATC

Commit message: vr input changed to lm1815
Parts:
- removed P11, P13, P16, P18, P51, P52: CONN_1, SIL-1, symbol CONN_1
- removed P4: CONN_25, symbol CONN_25
- added P1, P2: CONN_25X2, PIN_ARRAY_25x2_A, symbol CONN_25X2
- added P101: CONN_4, symbol CONN_4
- added P102, P103, P104, P105: CONN_1, symbol CONN_1
- added P106: CONN_6, symbol CONN_6
- added P107: CONN_10, symbol CONN_10
Connections:
- net 3.3V: now also P101.1 (P1), P2.5 (P5), P2.6 (P6)
- net 5V: now also P106.1, P107.1 (P1), P2.3 (P3), P2.4 (P4)
- net AN1-HARN: now also P107.9 (P9)
- net AN12-HARN: now also P107.2 (P2)
- net AN2-HARN: now also P107.8 (P8)
- net AN3-HARN: now also P107.7 (P7)
- net AN4-HARN: now also P107.6 (P6)
- net AN5-HARN: now also P107.5 (P5)
- net AN8-HARN: now also P107.4 (P4)
- net AN9-HARN: now also P107.3 (P3)
- net CAM+: now also P106.5
- net CAM-: now also P106.4
- net CRK2+: now also P106.2
- net CRK2-: now also P106.3
- net CPU-GND renamed GND
- net GND: now also P1.1 (P1), P1.2 (P2), P1.23 (P23), P1.49 (P49), P1.5 (P5), P1.50 (P50), P101.4 (P4), P102.1, P103.1, P104.1, P105.1, P106.6, P107.10 (P10), P2.1 (P1), P2.2 (P2), P2.49 (P49), P2.50 (P50)
- net stm32f407_board/PA5 renamed PA5
- net PA5: now also P1.15 (P15)
- net stm32f407_board/PC6 renamed PC6
- net PC6: now also P2.47 (P47)
- new net PA0: P1.12 (P12)
- new net PA1: P1.11 (P11)
- new net PA2: P1.14 (P14)
- new net PA3: P1.13 (P13)
- new net PA4: P1.16 (P16)
- new net PA6: P1.18 (P18)
- new net PA7: P1.17 (P17)
- new net PC1: P1.7 (P7)
- new net PC10: P101.3 (P3), P2.37 (P37)
- new net PC11: P101.2 (P2), P2.38 (P38)
- new net PC13: P2.12 (P12)
- new net PC2: P1.10 (P10)
- new net PC3: P1.9 (P9)
- new net PC4: P1.20 (P20)
- new net PC5: P1.19 (P19)
- new net PD7: P2.27 (P27)
- new net PE5: P2.14 (P14)
- new net PE6: P2.11 (P11)
- new net VDD: P1.3 (P3), P1.4 (P4)
- no-connect marks 16 -> 149
Other:
- note added: "Left conn"
- note added: "Right conn"
- note removed: "PB1 reset\ndefaults"
- note removed: "pg 10"
- moved on the sheet: C23, C24, D12, D13, D14, D15, JPO4, JPO5, P5, W23
